Commit message: Add the Robot Pkgs

File: src/description_pkg/urdf/description_pkg.urdf (robot description, URDF)
Before this commit: robot description_pkg, 4 links, 3 joints
Links:
- removed link lidar
- added link laser, mass 0.3304; collision mesh filename=package://description_pkg/meshes/lidar.STL; visual mesh filename=package://description_pkg/meshes/lidar.STL
Joints:
- joint joint_lidar: child lidar -> laser
